Commit message: added lidar dae file

File: gate-guider_ws/src/rect_bot_description_pkg/urdf/rect_bot.xacro (robot description, xacro)
@@ -85,5 +85,5 @@
       <origin xyz="0 0 0" rpy="0 0 0"/>
       <geometry>
-        <mesh filename="package://skbot_description/meshes/hokuyo.dae"/>
+        <mesh filename="package://rect_bot_description_pkg/meshes/hokuyo.dae"/>
       </geometry>
     </visual>

Commit message: added realsense camera onto robot model

File: gate-guider_ws/src/rect_bot_description_pkg/urdf/rect_bot.xacro (robot description, xacro)
@@ -40,30 +40,4 @@
         </visual>
     </link>
-  <!-- Adding a Camera -->
-  <joint name="joint_camera_base" type="fixed">
-    <parent link="chassis"/>
-    <child link="camera" />
-    <origin xyz="${chassisLength/2-cameraSize/2} 0 ${chassisHeight+wheelRadius}" rpy="0 0 0" />
-  </joint>
-  <link name="camera">
-    <collision>
-      <origin xyz="0 0 0" rpy="0 0 0"/>
-      <geometry>
-        <box size="${cameraSize} ${cameraSize} ${cameraSize}"/>
-      </geometry>
-    </collision>
-    <visual>
-      <origin xyz="0 0 0" rpy="0 0 0"/>
-      <geometry>
-        <box size="${cameraSize} ${cameraSize} ${cameraSize}"/>
-      </geometry>
-      <material name="blue"/>
-    </visual>
-    <inertial>
-      <mass value="${cameraMass}" />
-      <origin xyz="0 0 0" rpy="0 0 0"/>
-      <inertia ixx="0.000252666666667" ixy="0" ixz="0" iyy="0.000252666666667" iyz="0" izz="0.0005"/>
-    </inertial>
-  </link>
   <!-- Adding a Laser Scanner -->
   <joint name="joint_hokuyo" type="fixed">
@@ -94,3 +68,36 @@
     </inertial>
   </link>
+  <link name="front_realsense" />
+  <!--
+    The gazebo plugin aligns the depth data with the Z axis, with X=left and Y=up
+    ROS expects the depth data along the X axis, with Y=left and Z=up
+    This link only exists to give the gazebo plugin the correctly-oriented frame
+    -->
+  <link name="front_realsense_gazebo" />
+  <joint name="front_realsense_gazebo_joint" type="fixed">
+    <parent link="front_realsense"/>
+    <child link="front_realsense_gazebo"/>
+    <origin xyz="${chassisLength/2} 0 ${chassisHeight+wheelRadius+0.1}" rpy="-1.5707963267948966 0 -1.5707963267948966"/>
+  </joint>
+  <link name="front_realsense_lens">
+    <visual>
+      <origin xyz="0.02 0 0" rpy="${pi/2} 0 ${pi/2}" />
+      <geometry>
+        <mesh filename="package://realsense2_description/meshes/d435.dae" />
+      </geometry>
+      <material name="white" />
+    </visual>
+  </link>
+  <joint type="fixed" name="front_realsense_lens_joint">
+    <!-- Offset the camera 2cm backwards and 1cm up-->
+    <origin xyz="${chassisLength/2-0.02} 0 ${chassisHeight+wheelRadius+0.11}" rpy="0 0 0" />
+    <parent link="chassis" />
+    <child link="front_realsense_lens" />
+  </joint>
+  <joint type="fixed" name="front_realsense_joint">
+    <origin xyz="${chassisLength/2+0.025} 0 ${chassisHeight+wheelRadius+0.1}" rpy="0 0 0" />
+    <parent link="front_realsense_lens" />
+    <child link="front_realsense" />
+  </joint>
+  -->
 </robot>
